Commit message: adding the localization pkg

File: robot_description/urdf/robot_description.urdf.xacro (robot description, xacro)
@@ -140,3 +140,29 @@
     <axis xyz="0 0 0" />
   </joint>
+  <link name="imu_link">
+    <inertial>
+      <origin xyz="-0.00552433659106688 0.000168210391520346 0.000514000497342681" rpy="0 0 0" />
+      <mass value="0.000528415362211671" />
+      <inertia ixx="1.46176048428261E-08" ixy="1.40015117949421E-10" ixz="-1.99633872937403E-12"
+               iyy="8.59662482954888E-09" iyz="7.52375112767959E-12"
+               izz="2.30279421279312E-08" />
+    </inertial>
+    <visual>
+      <origin xyz="0.0 0.0 0.0" rpy="0.0 0.0 0.0"/>
+      <geometry>
+        <mesh filename="package://robot_description/meshes/imu_link.STL"/>
+      </geometry>
+    </visual>
+    <collision>
+      <origin xyz="0.0 0.0 0.0" rpy="0.0 0.0 0.0"/>
+      <geometry>
+        <mesh filename="package://robot_description/meshes/imu_link.STL"/>
+      </geometry>
+    </collision>
+  </link>
+  <joint name="imu_joint" type="fixed">
+    <origin xyz="0.0 0.0 0.07" rpy="0.0 0.0 0.0"/>
+    <parent link="base_link"/>
+    <child link="imu_link"/>
+  </joint>
 </robot>

File: robot_description/urdf/robot_description_gazebo.xacro (robot description, xacro)
@@ -57,4 +57,56 @@
     <maxVel>1.0</maxVel>
   </gazebo>
+  <!-- IMU -->
+  <gazebo reference="imu_link">
+    <sensor name="imu" type="imu">
+        <always_on>true</always_on>
+        <update_rate>100</update_rate>
+        <gz_frame_id>imu_link</gz_frame_id>
+        <topic>imu</topic>
+        <imu>
+          <angular_velocity>
+            <x>
+              <noise type="gaussian">
+                <mean>0.0</mean>
+                <stddev>2e-4</stddev>
+              </noise>
+            </x>
+            <y>
+              <noise type="gaussian">
+                <mean>0.0</mean>
+                <stddev>2e-4</stddev>
+              </noise>
+            </y>
+            <z>
+              <noise type="gaussian">
+                <mean>0.0</mean>
+                <stddev>2e-4</stddev>
+              </noise>
+            </z>
+          </angular_velocity>
+          <linear_acceleration>
+            <x>
+              <noise type="gaussian">
+                <mean>0.0</mean>
+                <stddev>1.7e-2</stddev>
+              </noise>
+            </x>
+            <y>
+              <noise type="gaussian">
+                <mean>0.0</mean>
+                <stddev>1.7e-2</stddev>
+              </noise>
+            </y>
+            <z>
+              <noise type="gaussian">
+                <mean>0.0</mean>
+                <stddev>1.7e-2</stddev>
+              </noise>
+            </z>
+          </linear_acceleration>
+        </imu>
+        <plugin name="imu" filename="libgazebo_ros_imu_sensor.so"/>
+    </sensor>
+  </gazebo>
   <gazebo>
     <plugin filename="libgazebo_ros2_control.so" name="gazebo_ros2_control">

Commit message: updating the localization pkg

File: robot_description/urdf/robot_description.urdf.xacro (robot description, xacro)
@@ -18,4 +18,5 @@
         <mesh filename="package://robot_description/meshes/base_link.STL" />
       </geometry>
+      <material name="red"/>
     </visual>
     <collision>
@@ -44,4 +45,5 @@
         <mesh filename="package://robot_description/meshes/right_wheel.STL" />
       </geometry>
+      <material name="blue"/>
     </visual>
     <collision>
@@ -72,4 +74,5 @@
         <mesh filename="package://robot_description/meshes/left_wheel.STL" />
       </geometry>
+      <material name="blue"/>
     </visual>
     <collision>
@@ -99,4 +102,5 @@
         <mesh filename="package://robot_description/meshes/front_caster.STL" />
       </geometry>
+      <material name="silver"/>
     </visual>
     <collision>
@@ -126,4 +130,5 @@
         <mesh filename="package://robot_description/meshes/rear_caster.STL" />
       </geometry>
+      <material name="silver"/>
     </visual>
     <collision>
@@ -153,4 +158,5 @@
         <mesh filename="package://robot_description/meshes/imu_link.STL"/>
       </geometry>
+      <material name="blue"/>
     </visual>
     <collision>
@@ -166,3 +172,15 @@
     <child link="imu_link"/>
   </joint>
+  <material name="blue">
+    <color rgba="0 0 1 1"/>
+  </material>
+  <material name="black">
+    <color rgba="0 0 0 1"/>
+  </material>
+  <material name="silver">
+    <color rgba="0.79 0.82 0.93 1"/>
+  </material>
+  <material name="dark_grey">
+    <color rgba="0.3 0.3 0.3 1"/>
+  </material>
 </robot>

Commit message: fixing controller manager error

File: robot_description/urdf/robot_description.urdf.xacro (robot description, xacro)
@@ -111,5 +111,5 @@
     </collision>
   </link>
-  <joint name="freont_caster_wheel_joint" type="fixed">
+  <joint name="front_caster_wheel_joint" type="fixed">
     <origin xyz="0.04755 0 -0.0275" rpy="0 0 0" />
     <parent link="base_link" />
@@ -172,4 +172,7 @@
     <child link="imu_link"/>
   </joint>
+  <material name="red">
+    <color rgba="1 0 0 1"/>
+  </material>
   <material name="blue">
     <color rgba="0 0 1 1"/>

File: robot_description/urdf/robot_description_gazebo.xacro (robot description, xacro)
@@ -110,8 +110,8 @@
   </gazebo>
   <gazebo>
-    <plugin filename="libgazebo_ros2_control.so" name="gazebo_ros2_control">
-      <robot_param>robot_description</robot_param>
-      <robot_param_node>robot_state_publisher</robot_param_node>
+    <plugin filename="ign_ros2_control-system" name="ign_ros2_control::IgnitionROS2ControlPlugin">
       <parameters>$(find robot_control)/config/robot_controllers.yaml</parameters>
+    </plugin>
+    <plugin filename="ignition-gazebo-imu-system" name="ignition::gazebo::systems::Imu">
     </plugin>
   </gazebo>

File: robot_description/urdf/robot_ros2_control.xacro (robot description, xacro)
@@ -3,5 +3,5 @@
     <ros2_control type="system" name="RobotSystem">
         <hardware>
-            <plugin>gazebo_ros2_control/GazeboSystem</plugin>
+            <plugin>ign_ros2_control/IgnitionSystem</plugin>
         </hardware>
         <joint name="right_wheel_joint">
